File: ADC_Board/ADC_Board_Right.brd (EAGLE design)
At the start: 63.5 x 81.3 mm, 24 parts

Commit message: Alterações ligeiras nos esquemas eléctricos das placas das ADCs.
Parts:
- renumbered JP11 to CON2_ADC_CS, JP12 to CON3_ADC_AGND, JP13 to CON4_ADC_SPI, JP14 to CON1_LED
Changed lines of the file:
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@@
 <element name="JP9" library="pinhead" package="1X06" value="" x="29.21" y="-53.34" rot="R90"/>
 <element name="JP10" library="pinhead" package="1X06" value="" x="34.29" y="-53.34" rot="R90"/>
-<element name="JP11" library="pinhead" package="2X03" value="" x="24.13" y="-68.58" smashed="yes">
-<attribute name="NAME" x="24.13" y="-74.93" size="1.27" layer="25" ratio="10" align="center"/>
+<element name="CON2_ADC_CS" library="pinhead" package="2X03" value="" x="24.13" y="-68.58" smashed="yes">
+<attribute name="NAME" x="24.13" y="-77.47" size="1.016" layer="25" ratio="10" align="center"/>
 <attribute name="VALUE" x="20.32" y="-73.025" size="1.27" layer="27"/>
 </element>
-<element name="JP12" library="pinhead" package="2X03" value="" x="39.37" y="-68.58" smashed="yes">
-<attribute name="NAME" x="39.37" y="-74.93" size="1.27" layer="25" ratio="10" align="center"/>
+<element name="CON3_ADC_AGND" library="pinhead" package="2X03" value="" x="39.37" y="-68.58" smashed="yes">
+<attribute name="NAME" x="38.1" y="-77.47" size="1.016" layer="25" ratio="10" align="center"/>
 <attribute name="VALUE" x="35.56" y="-73.025" size="1.27" layer="27"/>
 </element>
-<element name="JP13" library="pinhead" package="2X03" value="" x="54.61" y="-68.58" smashed="yes">
-<attribute name="NAME" x="54.61" y="-74.93" size="1.27" layer="25" ratio="10" align="center"/>
+<element name="CON4_ADC_SPI" library="pinhead" package="2X03" value="" x="54.61" y="-68.58" smashed="yes">
+<attribute name="NAME" x="52.07" y="-77.47" size="1.016" layer="25" ratio="10" align="center"/>
 <attribute name="VALUE" x="50.8" y="-73.025" size="1.27" layer="27"/>
 </element>
-<element name="JP14" library="pinhead" package="2X03" value="" x="8.89" y="-68.58" smashed="yes">
-<attribute name="NAME" x="8.89" y="-74.93" size="1.27" layer="25" ratio="10" align="center"/>
+<element name="CON1_LED" library="pinhead" package="2X03" value="" x="8.89" y="-68.58" smashed="yes">
+<attribute name="NAME" x="11.43" y="-77.47" size="1.016" layer="25" ratio="10" align="center"/>
 <attribute name="VALUE" x="5.08" y="-73.025" size="1.27" layer="27"/>
 </element>
@@
 </signal>
 <signal name="GND">
-<contactref element="JP14" pad="5"/>
-<contactref element="JP14" pad="6"/>
+<contactref element="CON1_LED" pad="5"/>
+<contactref element="CON1_LED" pad="6"/>
 <wire x1="11.43" y1="-69.85" x2="11.43" y2="-67.31" width="1.27" layer="16"/>
 <wire x1="11.43" y1="-59.69" x2="11.43" y2="-67.31" width="1.27" layer="16"/>
@@
 <contactref element="JP2" pad="2"/>
 <contactref element="JP1" pad="2"/>
-<contactref element="JP14" pad="3"/>
-<contactref element="JP14" pad="4"/>
+<contactref element="CON1_LED" pad="3"/>
+<contactref element="CON1_LED" pad="4"/>
 <wire x1="8.89" y1="-54.61" x2="8.89" y2="-69.85" width="1.27" layer="16"/>
 <wire x1="8.89" y1="-69.85" x2="8.89" y2="-67.31" width="1.27" layer="16"/>
@@
 <wire x1="46.99" y1="-36.83" x2="52.07" y2="-36.83" width="1.27" layer="16"/>
 <wire x1="52.07" y1="-36.83" x2="52.07" y2="-67.31" width="1.27" layer="16"/>
-<contactref element="JP13" pad="2"/>
+<contactref element="CON4_ADC_SPI" pad="2"/>
 </signal>
 <signal name="SCK">
@@
 <wire x1="46.99" y1="-31.75" x2="57.15" y2="-31.75" width="1.27" layer="16"/>
 <wire x1="57.15" y1="-31.75" x2="57.15" y2="-67.31" width="1.27" layer="16"/>
-<contactref element="JP13" pad="6"/>
+<contactref element="CON4_ADC_SPI" pad="6"/>
 </signal>
 <signal name="MISO">
@@
 <wire x1="46.99" y1="-34.29" x2="54.61" y2="-34.29" width="1.27" layer="16"/>
 <wire x1="54.61" y1="-34.29" x2="54.61" y2="-67.31" width="1.27" layer="16"/>
-<contactref element="JP13" pad="4"/>
+<contactref element="CON4_ADC_SPI" pad="4"/>
 </signal>
 <signal name="V+">
@@
 <wire x1="52.07" y1="-26.67" x2="59.69" y2="-26.67" width="1.27" layer="16"/>
 <wire x1="59.69" y1="-26.67" x2="59.69" y2="-69.85" width="1.27" layer="16"/>
-<contactref element="JP13" pad="5"/>
+<contactref element="CON4_ADC_SPI" pad="5"/>
 <wire x1="59.69" y1="-69.85" x2="57.15" y2="-69.85" width="1.27" layer="16"/>
 <contactref element="C1" pad="1"/>
-<contactref element="JP13" pad="3"/>
+<contactref element="CON4_ADC_SPI" pad="3"/>
 <wire x1="57.15" y1="-69.85" x2="54.61" y2="-69.85" width="1.27" layer="16"/>
-<contactref element="JP13" pad="1"/>
+<contactref element="CON4_ADC_SPI" pad="1"/>
 <wire x1="54.61" y1="-69.85" x2="52.07" y2="-69.85" width="1.27" layer="16"/>
 <wire x1="13.97" y1="-21.59" x2="46.99" y2="-21.59" width="1.27" layer="1"/>
@@
 <wire x1="44.45" y1="-49.53" x2="44.45" y2="-41.91" width="1.27" layer="16"/>
 <wire x1="44.45" y1="-41.91" x2="46.99" y2="-41.91" width="1.27" layer="16"/>
-<contactref element="JP12" pad="6"/>
+<contactref element="CON3_ADC_AGND" pad="6"/>
 <wire x1="41.91" y1="-67.31" x2="41.91" y2="-64.77" width="1.27" layer="16"/>
 <wire x1="41.91" y1="-64.77" x2="44.45" y2="-64.77" width="1.27" layer="16"/>
 <wire x1="44.45" y1="-64.77" x2="44.45" y2="-49.53" width="1.27" layer="16"/>
 <contactref element="C1" pad="2"/>
-<contactref element="JP12" pad="5"/>
+<contactref element="CON3_ADC_AGND" pad="5"/>
 <wire x1="44.45" y1="-29.21" x2="44.45" y2="-41.91" width="1.27" layer="16"/>
 <wire x1="41.91" y1="-67.31" x2="41.91" y2="-69.85" width="1.27" layer="16"/>
@@
 <contactref element="JP1" pad="3"/>
 <wire x1="3.81" y1="-13.97" x2="3.81" y2="-69.85" width="1.27" layer="16"/>
-<contactref element="JP14" pad="1"/>
+<contactref element="CON1_LED" pad="1"/>
 <wire x1="3.81" y1="-69.85" x2="6.35" y2="-69.85" width="1.27" layer="16"/>
 <wire x1="13.97" y1="-13.97" x2="3.81" y2="-13.97" width="1.27" layer="16"/>
@@
 <contactref element="JP6" pad="4"/>
 <wire x1="6.35" y1="-67.31" x2="6.35" y2="-52.07" width="1.27" layer="16"/>
-<contactref element="JP14" pad="2"/>
+<contactref element="CON1_LED" pad="2"/>
 <wire x1="6.35" y1="-52.07" x2="13.97" y2="-52.07" width="1.27" layer="16"/>
 </signal>
@@
 <wire x1="49.53" y1="-39.37" x2="49.53" y2="-72.39" width="1.27" layer="16"/>
 <wire x1="49.53" y1="-72.39" x2="39.37" y2="-72.39" width="1.27" layer="16"/>
-<contactref element="JP11" pad="1"/>
-<contactref element="JP11" pad="3"/>
-<contactref element="JP11" pad="5"/>
-<contactref element="JP11" pad="2"/>
-<contactref element="JP11" pad="4"/>
-<contactref element="JP11" pad="6"/>
-<contactref element="JP12" pad="1"/>
-<contactref element="JP12" pad="3"/>
-<contactref element="JP12" pad="2"/>
-<contactref element="JP12" pad="4"/>
+<contactref element="CON2_ADC_CS" pad="1"/>
+<contactref element="CON2_ADC_CS" pad="3"/>
+<contactref element="CON2_ADC_CS" pad="5"/>
+<contactref element="CON2_ADC_CS" pad="2"/>
+<contactref element="CON2_ADC_CS" pad="4"/>
+<contactref element="CON2_ADC_CS" pad="6"/>
+<contactref element="CON3_ADC_AGND" pad="1"/>
+<contactref element="CON3_ADC_AGND" pad="3"/>
+<contactref element="CON3_ADC_AGND" pad="2"/>
+<contactref element="CON3_ADC_AGND" pad="4"/>
 <wire x1="39.37" y1="-72.39" x2="36.83" y2="-72.39" width="1.27" layer="16"/>
 <wire x1="19.05" y1="-72.39" x2="24.13" y2="-72.39" width="1.27" layer="16"/>
